Commit message: add base link inertia

File: kuka_kr5_support/urdf/kr5_sixx_r650_macro.xacro (robot description, xacro)
@@ -6,4 +6,18 @@
     <link
     name="${prefix}base_link">
+    <inertial>
+      <origin
+        xyz="0.0 0.0 0.0"
+        rpy="0 0 0" />
+      <mass
+        value="5" />
+      <inertia
+        ixx="1.0"
+        ixy="0.0"
+        ixz="0.0"
+        iyy="1.0"
+        iyz="-0.0"
+        izz="1.0" />
+    </inertial>
     <visual>
       <origin
